Commit message: package added to store data and dummy script for publisghing the same

File: ensta_environments/ensta_gazebo_worlds/common/worlds/world-1.urdf.xacro (robot description, xacro)
@@ -32,11 +32,11 @@
 			<origin xyz="0 0 0" />
 			<geometry>
-				<box size="20 0.01 2.60" />
-			</geometry>
-		</visual>
-		<collision>
-			<origin xyz="0 0 0" />
-			<geometry>
-				<box size="20.02 0.03 2.62" />
+				<box size="20 0.50 2.60" />
+			</geometry>
+		</visual>
+		<collision>
+			<origin xyz="0 0 0" />
+			<geometry>
+				<box size="20.02 0.53 2.62" />
 			</geometry>
 		</collision>
@@ -57,11 +57,11 @@
 			<origin xyz="0 0 0" />
 			<geometry>
-				<box size="0.01 20 2.60" />
-			</geometry>
-		</visual>
-		<collision>
-			<origin xyz="0 0 0" />
-			<geometry>
-				<box size="0.03 20.02 2.62" />
+				<box size="0.50 20 2.60" />
+			</geometry>
+		</visual>
+		<collision>
+			<origin xyz="0 0 0" />
+			<geometry>
+				<box size="0.53 20.02 2.62" />
 			</geometry>
 		</collision>
@@ -82,11 +82,11 @@
 			<origin xyz="0 0 0" />
 			<geometry>
-				<box size="20 0.01 2.60" />
-			</geometry>
-		</visual>
-		<collision>
-			<origin xyz="0 0 0" />
-			<geometry>
-				<box size="20.2 0.03 2.62" />
+				<box size="20 0.50 2.60" />
+			</geometry>
+		</visual>
+		<collision>
+			<origin xyz="0 0 0" />
+			<geometry>
+				<box size="20.2 0.53 2.62" />
 			</geometry>
 		</collision>
@@ -107,11 +107,11 @@
 			<origin xyz="0 0 0" />
 			<geometry>
-				<box size="0.01 20 2.60" />
-			</geometry>
-		</visual>
-		<collision>
-			<origin xyz="0 0 0" />
-			<geometry>
-				<box size="0.03 20.02 2.62" />
+				<box size="0.50 20 2.60" />
+			</geometry>
+		</visual>
+		<collision>
+			<origin xyz="0 0 0" />
+			<geometry>
+				<box size="0.53 20.02 2.62" />
 			</geometry>
 		</collision>

Commit message: working first vesrion

File: ensta_environments/ensta_gazebo_worlds/common/worlds/world-1.urdf.xacro (robot description, xacro)
@@ -113,5 +113,5 @@
 			<origin xyz="0 0 0" />
 			<geometry>
-				<box size="0.53 20.02 2.62" />
+				<box size="0.52 20.02 2.62" />
 			</geometry>
 		</collision>
@@ -139,5 +139,5 @@
 			<origin xyz="-4 6 0" />
 			<geometry>
-				<box size="0.64 2.01 0.91" />
+				<box size="1.02 1.02 1.52" />
 			</geometry>
 		</collision>
@@ -146,5 +146,5 @@
 	</gazebo>
 	<joint name="joint_object_1" type="fixed">
-		<origin xyz="0 0 0.15" rpy="0 0 0" />
+		<origin xyz="0 0 0.45" rpy="0 0 0" />
 		<parent link="dummy_link" />
 		<child link="object_1" />
@@ -166,10 +166,10 @@
 			<origin xyz="-4 -6 0" />
 			<geometry>
-				<box size="0.64 2.01 0.91" />
+				<box size="1.02 1.02 1.52" />
 			</geometry>
 		</collision>
 	</link>
 	<joint name="joint_object_2" type="fixed">
-		<origin xyz="0 0 0.15" rpy="0 0 0" />
+		<origin xyz="0 0 0.45" rpy="0 0 0" />
 		<parent link="dummy_link" />
 		<child link="object_2" />
@@ -191,10 +191,10 @@
 			<origin xyz="5 0 0" />
 			<geometry>
-				<box size="0.64 2.01 0.91" />
+				<box size="1.02 1.02 1.52" />
 			</geometry>
 		</collision>
 	</link>
 	<joint name="joint_object_3" type="fixed">
-		<origin xyz="0 0 0.15" rpy="0 0 0" />
+		<origin xyz="0 0 0.45" rpy="0 0 0" />
 		<parent link="dummy_link" />
 		<child link="object_3" />

File: ensta_environments/ensta_gazebo_worlds/common/worlds/world-2.urdf.xacro (robot description, xacro)
@@ -122,4 +122,157 @@
 		<child link="west_wall" />
 	</joint>
+        <!-- center_wall_one -->
+	<link name="center_wall_one">
+		<inertial>
+			<origin xyz="0 0 0" />
+			<mass value="5.0" />
+			<inertia ixx="0.0" ixy="0.0" ixz="0.0" iyy="0.0" iyz="0.0" izz="0.0" />
+		</inertial>
+		<visual>
+			<origin xyz="0 0 0" />
+			<geometry>
+				<box size="10 0.01 2.60" />
+			</geometry>
+		</visual>
+		<collision>
+			<origin xyz="0 0 0" />
+			<geometry>
+				<box size="10.02 0.03 2.62" />
+			</geometry>
+		</collision>
+	</link>
+	<joint name="joint_center_wall_one" type="fixed">
+		<origin xyz="-5 2 1" rpy="0 0 0" />
+		<parent link="dummy_link" />
+		<child link="center_wall_one" />
+	</joint>
+        <!-- center_wall_two -->
+	<link name="center_wall_two">
+		<inertial>
+			<origin xyz="0 0 0" />
+			<mass value="5.0" />
+			<inertia ixx="0.0" ixy="0.0" ixz="0.0" iyy="0.0" iyz="0.0" izz="0.0" />
+		</inertial>
+		<visual>
+			<origin xyz="0 0 0" />
+			<geometry>
+				<box size="9 0.01 2.60" />
+			</geometry>
+		</visual>
+		<collision>
+			<origin xyz="0 0 0" />
+			<geometry>
+				<box size="9.02 0.03 2.62" />
+			</geometry>
+		</collision>
+	</link>
+	<joint name="joint_center_wall_two" type="fixed">
+		<origin xyz="5.5 2 1" rpy="0 0 0" />
+		<parent link="dummy_link" />
+		<child link="center_wall_two" />
+	</joint>
+<!-- Objects -->
+	<!-- object_1 -->
+	<link name="object_1">
+		<inertial>
+			<origin xyz="-4 6 0" />
+			<mass value="5.0" />
+			<inertia ixx="0.0" ixy="0.0" ixz="0.0" iyy="0.0" iyz="0.0" izz="0.0" />
+		</inertial>
+		<visual>
+			<origin xyz="-4 6 0" />
+			<geometry>
+				<box size="1 1 1.5" />
+			</geometry>
+		</visual>
+		<collision>
+			<origin xyz="-4 6 0" />
+			<geometry>
+				<box size="1.02 1.02 1.52" />
+			</geometry>
+		</collision>
+	</link>
+	<gazebo reference="object_1">
+	</gazebo>
+	<joint name="joint_object_1" type="fixed">
+		<origin xyz="0 0 0.45" rpy="0 0 0" />
+		<parent link="dummy_link" />
+		<child link="object_1" />
+	</joint>
+	<!-- object_2 -->
+	<link name="object_2">
+		<inertial>
+			<origin xyz="-4 0 0" />
+			<mass value="5.0" />
+			<inertia ixx="0.0" ixy="0.0" ixz="0.0" iyy="0.0" iyz="0.0" izz="0.0" />
+		</inertial>
+		<visual>
+			<origin xyz="-4 0 0" />
+			<geometry>
+				<box size="1 1 1.5" />
+			</geometry>
+		</visual>
+		<collision>
+			<origin xyz="-4 0 0" />
+			<geometry>
+				<box size="1.02 1.02 1.52" />
+			</geometry>
+		</collision>
+	</link>
+	<joint name="joint_object_2" type="fixed">
+		<origin xyz="0 0 0.45" rpy="0 0 0" />
+		<parent link="dummy_link" />
+		<child link="object_2" />
+	</joint>
+	<!-- object_3 -->
+	<link name="object_3">
+		<inertial>
+			<origin xyz="5 0 0" />
+			<mass value="5.0" />
+			<inertia ixx="0.0" ixy="0.0" ixz="0.0" iyy="0.0" iyz="0.0" izz="0.0" />
+		</inertial>
+		<visual>
+			<origin xyz="5 0 0" />
+			<geometry>
+				<box size="1 1 1.5" />
+			</geometry>
+		</visual>
+		<collision>
+			<origin xyz="5 0 0" />
+			<geometry>
+				<box size="1.02 1.02 1.52" />
+			</geometry>
+		</collision>
+	</link>
+	<joint name="joint_object_3" type="fixed">
+		<origin xyz="0 0 0.45" rpy="0 0 0" />
+		<parent link="dummy_link" />
+		<child link="object_3" />
+	</joint>
+        <!-- object_4 -->
+	<link name="object_4">
+		<inertial>
+			<origin xyz="-4 -6 0" />
+			<mass value="5.0" />
+			<inertia ixx="0.0" ixy="0.0" ixz="0.0" iyy="0.0" iyz="0.0" izz="0.0" />
+		</inertial>
+		<visual>
+			<origin xyz="-4 -6 0" />
+			<geometry>
+				<box size="1 1 1.5" />
+			</geometry>
+		</visual>
+		<collision>
+			<origin xyz="-4 -6 0" />
+			<geometry>
+				<box size="1.02 1.02 1.52" />
+			</geometry>
+		</collision>
+	</link>
+	<joint name="joint_object_4" type="fixed">
+		<origin xyz="0 0 0.45" rpy="0 0 0" />
+		<parent link="dummy_link" />
+		<child link="object_4" />
+	</joint>
  <gazebo reference="north_wall">
 	<material>Gazebo/White</material>
@@ -138,3 +291,27 @@
 	<selfCollide>false</selfCollide>
  </gazebo>
+ <gazebo reference="center_wall_one">
+	<material>Gazebo/White</material>
+	<selfCollide>false</selfCollide>
+ </gazebo>
+ <gazebo reference="center_wall_two">
+	<material>Gazebo/White</material>
+	<selfCollide>false</selfCollide>
+ </gazebo>
+ <gazebo reference="object_1">
+	<material>Gazebo/Blue</material>
+	<selfCollide>false</selfCollide>
+ </gazebo>
+ <gazebo reference="object_2">
+	<material>Gazebo/Blue</material>
+	<selfCollide>false</selfCollide>
+ </gazebo>
+ <gazebo reference="object_3">
+	<material>Gazebo/Blue</material>
+	<selfCollide>false</selfCollide>
+ </gazebo>
+ <gazebo reference="object_4">
+	<material>Gazebo/Blue</material>
+	<selfCollide>false</selfCollide>
+ </gazebo>
 </robot>

File: ensta_robots/urdf/pioneer3dx.xacro (robot description, xacro)
@@ -394,5 +394,5 @@
 				<range>
 					<min>0.10</min>
-					<max>30.0</max>
+					<max>4.0</max>
 					<resolution>0.01</resolution>
 				</range>
