Commit message: created a test scenario

File: ensta_environments/ensta_gazebo_objects/common/objects/heavy_object.urdf.xacro (robot description, xacro)
@@ -8,13 +8,13 @@
      </inertial>
      <visual>
-       <origin xyz="0 0 0"/>
+       <origin xyz="0 -0.1 0"/>
        <geometry>
-         <box size="1.5 1.5 0.9" />
+         <mesh filename="package://ensta_gazebo_objects/Media/materials/textures/stool.dae" />
        </geometry>
      </visual>
      <collision>
-       <origin xyz="0 0 0"/>
+       <origin xyz="0 0. 0"/>
        <geometry>
-         <box size="1.5 1.5 0.9" />
+         <box size="0.2 0.2 0.2" />
        </geometry>
      </collision>

File: ensta_environments/ensta_gazebo_worlds/common/worlds/world-3.urdf.xacro (robot description, xacro)
@@ -1,4 +1,4 @@
 <?xml version="1.0"?>
-<robot name="demo-3">
+<robot name="demo-1">
 	<!-- dummy_link -->
 	<link name="dummy_link">
@@ -32,5 +32,5 @@
 			<origin xyz="0 0 0" />
 			<geometry>
-				<box size="20 0.01 2.60" />
+				<box size="14 0.01 1.5" />
 			</geometry>
 		</visual>
@@ -38,5 +38,5 @@
 			<origin xyz="0 0 0" />
 			<geometry>
-				<box size="20.02 0.03 2.62" />
+				<box size="14.02 0.03 1.62" />
 			</geometry>
 		</collision>
@@ -122,6 +122,56 @@
 		<child link="west_wall" />
 	</joint>
+        <!-- center_wall_one -->
+	<link name="center_wall_one">
+		<inertial>
+			<origin xyz="0 0 0" />
+			<mass value="5.0" />
+			<inertia ixx="0.0" ixy="0.0" ixz="0.0" iyy="0.0" iyz="0.0" izz="0.0" />
+		</inertial>
+		<visual>
+			<origin xyz="0 0 0" />
+			<geometry>
+				<box size="10 0.01 2.60" />
+			</geometry>
+		</visual>
+		<collision>
+			<origin xyz="0 0 0" />
+			<geometry>
+				<box size="10.02 0.03 2.62" />
+			</geometry>
+		</collision>
+	</link>
+	<joint name="joint_center_wall_one" type="fixed">
+		<origin xyz="-5 2 1" rpy="0 0 0" />
+		<parent link="dummy_link" />
+		<child link="center_wall_one" />
+	</joint>
+        <!-- center_wall_two -->
+	<link name="center_wall_two">
+		<inertial>
+			<origin xyz="0 0 0" />
+			<mass value="5.0" />
+			<inertia ixx="0.0" ixy="0.0" ixz="0.0" iyy="0.0" iyz="0.0" izz="0.0" />
+		</inertial>
+		<visual>
+			<origin xyz="0 0 0" />
+			<geometry>
+				<box size="9 0.01 2.60" />
+			</geometry>
+		</visual>
+		<collision>
+			<origin xyz="0 0 0" />
+			<geometry>
+				<box size="9.02 0.03 2.62" />
+			</geometry>
+		</collision>
+	</link>
+	<joint name="joint_center_wall_two" type="fixed">
+		<origin xyz="5.5 2 1" rpy="0 0 0" />
+		<parent link="dummy_link" />
+		<child link="center_wall_two" />
+	</joint>
  <gazebo reference="north_wall">
-	<material>Gazebo/White</material>
+	<material>IPA/Wall2</material>
 	<selfCollide>false</selfCollide>
  </gazebo>
@@ -138,3 +188,11 @@
 	<selfCollide>false</selfCollide>
  </gazebo>
+ <gazebo reference="center_wall_one">
+	<material>Gazebo/White</material>
+	<selfCollide>false</selfCollide>
+ </gazebo>
+ <gazebo reference="center_wall_two">
+	<material>Gazebo/White</material>
+	<selfCollide>false</selfCollide>
+ </gazebo>
 </robot>
