Commit message: made changes in cob_simulation, ensta_gazebo_objects, robocup packages urdf files to make the scenario_1 work.

File: ensta_environments/ensta_gazebo_objects/common/objects/corrogated_box.urdf (robot description, URDF)
Before this commit: robot my_object, 1 links, 0 joints
Links:
- link base_link: mass 0.100 -> 0.05

File: ensta_environments/ensta_gazebo_objects/common/objects/corrogated_box_two.urdf (robot description, URDF)
Before this commit: robot my_object, 1 links, 0 joints
Links:
- link base_link: geometry collision mesh filename=package://ensta_gazebo_objects/Media/models/corrogated_box.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 scale=1.5 1.5 2.0; visual mesh filename=package://ensta_gazebo_objects/Media/models/corrogated_box.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 scale=1.5 1.5 2.0

File: ensta_environments/ensta_gazebo_objects/common/objects/stool.urdf (robot description, URDF)
Before this commit: robot stool, 1 links, 0 joints
Links:
- link stool: mass 1.0 -> 0.05
